File: tinyevse.sch (KiCad schematic (older format))
At the start: 11 parts

Commit message: add ICSP programming connector
Parts:
- added P?: ICSP, symbol CONN_02X03
Connections:
- net labels added: PWM, miso, mosi, sck
Other:
- moved on the sheet: X?
Changed lines of the file:
@@
 L RESONATOR X?
 U 1 1 571573AA
-P 5900 3200
-F 0 "X?" H 5900 3350 60  0000 C CNN
-F 1 "16MHz" H 5900 3050 60  0000 C CNN
-F 2 "" H 5900 3200 60  0000 C CNN
-F 3 "" H 5900 3200 60  0000 C CNN
-	1    5900 3200
+P 6000 3200
+F 0 "X?" H 6000 3350 60  0000 C CNN
+F 1 "16MHz" H 6000 3050 60  0000 C CNN
+F 2 "" H 6000 3200 60  0000 C CNN
+F 3 "" H 6000 3200 60  0000 C CNN
+	1    6000 3200
 	0    -1   -1   0
 $EndComp
 Wire Wire Line
-	5900 2900 5700 2900
-Wire Wire Line
-	5700 2900 5700 3150
-Wire Wire Line
-	5700 3150 5500 3150
-Wire Wire Line
-	5500 3250 5700 3250
-Wire Wire Line
-	5700 3250 5700 3500
-Wire Wire Line
-	5700 3500 5900 3500
+	6000 2900 5800 2900
+Wire Wire Line
+	5800 2900 5800 3150
+Wire Wire Line
+	5800 3150 5500 3150
+Wire Wire Line
+	5500 3250 5800 3250
+Wire Wire Line
+	5800 3250 5800 3500
+Wire Wire Line
+	5800 3500 6000 3500
 $Comp
 L GND #PWR?
 U 1 1 57157477
-P 6250 3200
-F 0 "#PWR?" H 6250 2950 50  0001 C CNN
-F 1 "GND" H 6250 3050 50  0000 C CNN
-F 2 "" H 6250 3200 50  0000 C CNN
-F 3 "" H 6250 3200 50  0000 C CNN
-	1    6250 3200
+P 6350 3200
+F 0 "#PWR?" H 6350 2950 50  0001 C CNN
+F 1 "GND" H 6350 3050 50  0000 C CNN
+F 2 "" H 6350 3200 50  0000 C CNN
+F 3 "" H 6350 3200 50  0000 C CNN
+	1    6350 3200
 	1    0    0    -1
 $EndComp
@@
 	1    0    0    -1
 $EndComp
+Text Label 5500 2550 0    60   ~ 0
+PWM
+Text Label 6300 4150 2    60   ~ 0
+PWM
+$Comp
+L CONN_02X03 P?
+U 1 1 57157DFA
+P 3050 4800
+F 0 "P?" H 3050 5000 50  0000 C CNN
+F 1 "ICSP" H 3050 4600 50  0000 C CNN
+F 2 "" H 3050 3600 50  0000 C CNN
+F 3 "" H 3050 3600 50  0000 C CNN
+	1    3050 4800
+	1    0    0    -1
+$EndComp
+Text Label 2800 4700 2    60   ~ 0
+miso
+Text Label 2800 4800 2    60   ~ 0
+sck
+Text Label 2800 4900 2    60   ~ 0
+reset
+$Comp
+L VDD #PWR?
+U 1 1 57157FD2
+P 3300 4700
+F 0 "#PWR?" H 3300 4550 50  0001 C CNN
+F 1 "VDD" H 3300 4850 50  0000 C CNN
+F 2 "" H 3300 4700 50  0000 C CNN
+F 3 "" H 3300 4700 50  0000 C CNN
+	1    3300 4700
+	1    0    0    -1
+$EndComp
+$Comp
+L GND #PWR?
+U 1 1 57157FFE
+P 3300 4900
+F 0 "#PWR?" H 3300 4650 50  0001 C CNN
+F 1 "GND" H 3300 4750 50  0000 C CNN
+F 2 "" H 3300 4900 50  0000 C CNN
+F 3 "" H 3300 4900 50  0000 C CNN
+	1    3300 4900
+	1    0    0    -1
+$EndComp
+Text Label 3300 4800 0    60   ~ 0
+mosi
+Text Label 5500 3050 0    60   ~ 0
+sck
+Text Label 5500 2950 0    60   ~ 0
+miso
+Text Label 5500 2850 0    60   ~ 0
+mosi
 $EndSCHEMATC

Commit message: add a lot of stuff, move PWM pin
Parts:
- added C?: 104, symbol C
- added C?: 100uF, symbol CAPAPOL
- added D6: 1N4148, symbol D
- added D?: 13V ZENER, symbol ZENER
- added D?: 1N4007, symbol D
- added K?: RELAY, symbol RELAY_2RT
- added P?: Pilot, symbol CONN_01X03
- added R1: 650, symbol R
- added R2: 10K, symbol R
- added R3: 1K, symbol R
- added R5: 56K, symbol R
- added R6: 100K, symbol R
- added R7: 200K, symbol R
- C?: value C -> 104
Connections:
- net labels added: AMP_READ, PILOT, PILOTREAD, PP, PP_READ, RELAY, RELAY_COIL
- wire segments 14 -> 33
Other:
- note added: "+12V"
- note added: "+5V"
- moved on the sheet: C?, R?, SW?, U?A, X?

Commit message: annotate and add proper footprints to all but relay
Parts:
- added D1: D, Diodes_ThroughHole:Diode_DO-41_SOD81_Horizontal_RM10, symbol D
- added P2: 12V input, battery-dlg:CCFLHV, symbol CONN_01X02
- C1, C2, C4, C6: renamed from C?; footprint (none) -> Capacitors_ThroughHole:C_Rect_L7_W2.5_P5
- C3, C5: renamed from C?; footprint (none) -> Capacitors_ThroughHole:C_Radial_D7.5_L11.2_P2.5
- D2, D3: renamed from D?; footprint (none) -> Diodes_ThroughHole:Diode_DO-41_SOD81_Horizontal_RM10
- D6: footprint (none) -> Diodes_ThroughHole:Diode_DO-35_SOD27_Horizontal_RM10
- IC1: renamed from IC?; footprint DIL28 -> Housings_DIP:DIP-28_W7.62mm_LongPads
- P1: renamed from P?; footprint (none) -> Pin_Headers:Pin_Header_Straight_1x06
- P3: renamed from P?; footprint (none) -> Pin_Headers:Pin_Header_Straight_2x03
- P4: renamed from P?; footprint (none) -> Connect:PINHEAD1-3
- R1, R2, R3, R5, R6, R7: footprint (none) -> Resistors_ThroughHole:Resistor_Horizontal_RM10mm
- R10: renamed from R?; footprint (none) -> Resistors_ThroughHole:Resistor_Horizontal_RM10mm
- SW1: renamed from SW?; footprint (none) -> battery-dlg:SW-1825027-5
- U1: renamed from U?; footprint (none) -> battery-dlg:TO220_7805
- U2: renamed from U?; footprint (none) -> Power_Integrations:PDIP-8
- X1: renamed from X?; footprint (none) -> battery-dlg:HC-49V-OR-RESONATOR
- gave numbers to parts that had none: 1
Connections:
- wire segments 33 -> 35

Commit message: board is well underway
Connections:
- wire segments 35 -> 36
Other:
- moved on the sheet: C1, P1, P3
Changed lines of the file:
@@
 Text Label 5500 4000 0    60   ~ 0
 reset
-Text Label 3200 2250 2    60   ~ 0
+Text Label 3200 3000 2    60   ~ 0
 reset
 $Comp
@@
 L CONN_6 P1
 U 1 1 5715784B
-P 2750 3850
-F 0 "P1" V 2700 3850 60  0000 C CNN
-F 1 "SERIAL" V 2800 3850 60  0000 C CNN
-F 2 "Pin_Headers:Pin_Header_Straight_1x06" H 2750 3850 60  0001 C CNN
-F 3 "" H 2750 3850 60  0000 C CNN
-	1    2750 3850
+P 2850 3700
+F 0 "P1" V 2800 3700 60  0000 C CNN
+F 1 "SERIAL" V 2900 3700 60  0000 C CNN
+F 2 "Pin_Headers:Pin_Header_Straight_1x06" H 2850 3700 60  0001 C CNN
+F 3 "" H 2850 3700 60  0000 C CNN
+	1    2850 3700
 	-1   0    0    1
 $EndComp
@@
 L GND #PWR07
 U 1 1 571578E0
-P 3100 4150
-F 0 "#PWR07" H 3100 3900 50  0001 C CNN
-F 1 "GND" H 3100 4000 50  0000 C CNN
-F 2 "" H 3100 4150 50  0000 C CNN
-F 3 "" H 3100 4150 50  0000 C CNN
-	1    3100 4150
-	1    0    0    -1
-$EndComp
-Wire Wire Line
-	3100 4150 3100 4000
-Wire Wire Line
-	3250 3900 3100 3900
-Text Label 3150 3700 0    60   ~ 0
+P 3200 4000
+F 0 "#PWR07" H 3200 3750 50  0001 C CNN
+F 1 "GND" H 3200 3850 50  0000 C CNN
+F 2 "" H 3200 4000 50  0000 C CNN
+F 3 "" H 3200 4000 50  0000 C CNN
+	1    3200 4000
+	1    0    0    -1
+$EndComp
+Wire Wire Line
+	3200 4000 3200 3850
+Wire Wire Line
+	3350 3750 3200 3750
+Text Label 3250 3550 0    60   ~ 0
 TX
-Text Label 3150 3800 0    60   ~ 0
+Text Label 3250 3650 0    60   ~ 0
 RX
 Wire Wire Line
-	3150 3800 3100 3800
-Wire Wire Line
-	3100 3700 3150 3700
-Text Label 3100 3300 0    60   ~ 0
-reset
+	3250 3650 3200 3650
+Wire Wire Line
+	3200 3550 3250 3550
 $Comp
 L C C1
 U 1 1 571579E5
-P 3100 3450
-F 0 "C1" H 3125 3550 50  0000 L CNN
-F 1 "104" H 3125 3350 50  0000 L CNN
-F 2 "Capacitors_ThroughHole:C_Rect_L7_W2.5_P5" H 3138 3300 50  0001 C CNN
-F 3 "" H 3100 3450 50  0000 C CNN
-	1    3100 3450
+P 3200 3150
+F 0 "C1" H 3225 3250 50  0000 L CNN
+F 1 "104" H 3225 3050 50  0000 L CNN
+F 2 "Capacitors_ThroughHole:C_Rect_L7_W2.5_P5" H 3238 3000 50  0001 C CNN
+F 3 "" H 3200 3150 50  0000 C CNN
+	1    3200 3150
 	1    0    0    -1
 $EndComp
@@
 L VDD #PWR09
 U 1 1 57157BE7
-P 3250 3900
-F 0 "#PWR09" H 3250 3750 50  0001 C CNN
-F 1 "VDD" H 3250 4050 50  0000 C CNN
-F 2 "" H 3250 3900 50  0000 C CNN
-F 3 "" H 3250 3900 50  0000 C CNN
-	1    3250 3900
+P 3350 3750
+F 0 "#PWR09" H 3350 3600 50  0001 C CNN
+F 1 "VDD" H 3350 3900 50  0000 C CNN
+F 2 "" H 3350 3750 50  0000 C CNN
+F 3 "" H 3350 3750 50  0000 C CNN
+	1    3350 3750
 	-1   0    0    1
 $EndComp
@@
 L CONN_02X03 P3
 U 1 1 57157DFA
-P 3050 4800
-F 0 "P3" H 3050 5000 50  0000 C CNN
-F 1 "ICSP" H 3050 4600 50  0000 C CNN
-F 2 "Pin_Headers:Pin_Header_Straight_2x03" H 3050 3600 50  0001 C CNN
-F 3 "" H 3050 3600 50  0000 C CNN
-	1    3050 4800
-	1    0    0    -1
-$EndComp
-Text Label 2800 4700 2    60   ~ 0
+P 3050 4650
+F 0 "P3" H 3050 4850 50  0000 C CNN
+F 1 "ICSP" H 3050 4450 50  0000 C CNN
+F 2 "Pin_Headers:Pin_Header_Straight_2x03" H 3050 3450 50  0001 C CNN
+F 3 "" H 3050 3450 50  0000 C CNN
+	1    3050 4650
+	1    0    0    -1
+$EndComp
+Text Label 2800 4550 2    60   ~ 0
 miso
-Text Label 2800 4800 2    60   ~ 0
+Text Label 2800 4650 2    60   ~ 0
 sck
-Text Label 2800 4900 2    60   ~ 0
+Text Label 2800 4750 2    60   ~ 0
 reset
 $Comp
 L VDD #PWR015
 U 1 1 57157FD2
-P 3300 4700
-F 0 "#PWR015" H 3300 4550 50  0001 C CNN
-F 1 "VDD" H 3300 4850 50  0000 C CNN
-F 2 "" H 3300 4700 50  0000 C CNN
-F 3 "" H 3300 4700 50  0000 C CNN
-	1    3300 4700
+P 3300 4550
+F 0 "#PWR015" H 3300 4400 50  0001 C CNN
+F 1 "VDD" H 3300 4700 50  0000 C CNN
+F 2 "" H 3300 4550 50  0000 C CNN
+F 3 "" H 3300 4550 50  0000 C CNN
+	1    3300 4550
 	1    0    0    -1
 $EndComp
@@
 L GND #PWR016
 U 1 1 57157FFE
-P 3300 4900
-F 0 "#PWR016" H 3300 4650 50  0001 C CNN
-F 1 "GND" H 3300 4750 50  0000 C CNN
-F 2 "" H 3300 4900 50  0000 C CNN
-F 3 "" H 3300 4900 50  0000 C CNN
-	1    3300 4900
-	1    0    0    -1
-$EndComp
-Text Label 3300 4800 0    60   ~ 0
+P 3300 4750
+F 0 "#PWR016" H 3300 4500 50  0001 C CNN
+F 1 "GND" H 3300 4600 50  0000 C CNN
+F 2 "" H 3300 4750 50  0000 C CNN
+F 3 "" H 3300 4750 50  0000 C CNN
+	1    3300 4750
+	1    0    0    -1
+$EndComp
+Text Label 3300 4650 0    60   ~ 0
 mosi
 Text Label 5500 3050 0    60   ~ 0
@@
 	3250 2550 3200 2550
 Wire Wire Line
-	3200 2550 3200 2250
+	3200 2550 3200 3000
 $Comp
 L D D2
@@
 Wire Wire Line
 	3250 1750 3150 1750
+Wire Wire Line
+	3200 3300 3200 3450
 $EndSCHEMATC

Commit message: had the wrong footprint for 104 capacitors
Parts:
- C1, C2, C4, C6: footprint Capacitors_ThroughHole:C_Rect_L7_W2.5_P5 -> Capacitors_ThroughHole:C_Disc_D3_P2.5
Changed lines of the file:
@@
 F 0 "C2" H 3625 3400 50  0000 L CNN
 F 1 "104" H 3450 3200 50  0000 L CNN
-F 2 "Capacitors_ThroughHole:C_Rect_L7_W2.5_P5" H 3638 3150 50  0001 C CNN
+F 2 "Capacitors_ThroughHole:C_Disc_D3_P2.5" H 3638 3150 50  0001 C CNN
 F 3 "" H 3600 3300 50  0000 C CNN
 	1    3600 3300
@@
 F 0 "C6" H 5575 1900 50  0000 L CNN
 F 1 "104" H 5575 1700 50  0000 L CNN
-F 2 "Capacitors_ThroughHole:C_Rect_L7_W2.5_P5" H 5588 1650 50  0001 C CNN
+F 2 "Capacitors_ThroughHole:C_Disc_D3_P2.5" H 5588 1650 50  0001 C CNN
 F 3 "" H 5550 1800 50  0000 C CNN
 	1    5550 1800
@@
 F 0 "C1" H 3225 3250 50  0000 L CNN
 F 1 "104" H 3225 3050 50  0000 L CNN
-F 2 "Capacitors_ThroughHole:C_Rect_L7_W2.5_P5" H 3238 3000 50  0001 C CNN
+F 2 "Capacitors_ThroughHole:C_Disc_D3_P2.5" H 3238 3000 50  0001 C CNN
 F 3 "" H 3200 3150 50  0000 C CNN
 	1    3200 3150
@@
 F 0 "C4" H 4425 1950 50  0000 L CNN
 F 1 "104" H 4425 1750 50  0000 L CNN
-F 2 "Capacitors_ThroughHole:C_Rect_L7_W2.5_P5" H 4438 1700 50  0001 C CNN
+F 2 "Capacitors_ThroughHole:C_Disc_D3_P2.5" H 4438 1700 50  0001 C CNN
 F 3 "" H 4400 1850 50  0000 C CNN
 	1    4400 1850

Commit message: add 2-pin connector for external relay coil
Parts:
- added P5: RELAYCOIL, battery-dlg:CCFLHV, symbol CONN_01X02
- D1: value D -> 1N4007
Connections:
- wire segments 36 -> 37
Changed lines of the file:
@@
 LIBS:valves
 LIBS:arbduino-cache
-LIBS:tinyevse-cache
 EELAYER 25 0
 EELAYER END
@@
 $EndComp
 $Comp
-L GND #PWR01
+L GND #PWR9
 U 1 1 5715724D
 P 3600 4950
-F 0 "#PWR01" H 3600 4700 50  0001 C CNN
+F 0 "#PWR9" H 3600 4700 50  0001 C CNN
 F 1 "GND" H 3600 4800 50  0000 C CNN
 F 2 "" H 3600 4950 50  0000 C CNN
@@
 $EndComp
 $Comp
-L GND #PWR02
+L GND #PWR8
 U 1 1 571572BC
 P 3600 3450
-F 0 "#PWR02" H 3600 3200 50  0001 C CNN
+F 0 "#PWR8" H 3600 3200 50  0001 C CNN
 F 1 "GND" H 3600 3300 50  0000 C CNN
 F 2 "" H 3600 3450 50  0000 C CNN
@@
 Connection ~ 3600 2550
 $Comp
-L GND #PWR03
+L GND #PWR16
 U 1 1 5715733B
 P 5550 1950
-F 0 "#PWR03" H 5550 1700 50  0001 C CNN
+F 0 "#PWR16" H 5550 1700 50  0001 C CNN
 F 1 "GND" H 5550 1800 50  0000 C CNN
 F 2 "" H 5550 1950 50  0000 C CNN
@@
 	6050 3250 6300 3500
 $Comp
-L GND #PWR04
+L GND #PWR18
 U 1 1 57157477
 P 6650 3200
-F 0 "#PWR04" H 6650 2950 50  0001 C CNN
+F 0 "#PWR18" H 6650 2950 50  0001 C CNN
 F 1 "GND" H 6650 3050 50  0000 C CNN
 F 2 "" H 6650 3200 50  0000 C CNN
@@
 $EndComp
 $Comp
-L GND #PWR05
+L GND #PWR15
 U 1 1 571574DF
 P 5200 2050
-F 0 "#PWR05" H 5200 1800 50  0001 C CNN
+F 0 "#PWR15" H 5200 1800 50  0001 C CNN
 F 1 "GND" H 5200 1900 50  0000 C CNN
 F 2 "" H 5200 2050 50  0000 C CNN
@@
 $EndComp
 $Comp
-L GND #PWR06
+L GND #PWR1
 U 1 1 571576F7
 P 2600 2750
-F 0 "#PWR06" H 2600 2500 50  0001 C CNN
+F 0 "#PWR1" H 2600 2500 50  0001 C CNN
 F 1 "GND" H 2600 2600 50  0000 C CNN
 F 2 "" H 2600 2750 50  0000 C CNN
@@
 $EndComp
 $Comp
-L GND #PWR07
+L GND #PWR2
 U 1 1 571578E0
 P 3200 4000
-F 0 "#PWR07" H 3200 3750 50  0001 C CNN
+F 0 "#PWR2" H 3200 3750 50  0001 C CNN
 F 1 "GND" H 3200 3850 50  0000 C CNN
 F 2 "" H 3200 4000 50  0000 C CNN
@@
 $EndComp
 $Comp
-L VDD #PWR08
+L VDD #PWR7
 U 1 1 57157BA5
 P 3600 2500
-F 0 "#PWR08" H 3600 2350 50  0001 C CNN
+F 0 "#PWR7" H 3600 2350 50  0001 C CNN
 F 1 "VDD" H 3600 2650 50  0000 C CNN
 F 2 "" H 3600 2500 50  0000 C CNN
@@
 $EndComp
 $Comp
-L VDD #PWR09
+L VDD #PWR6
 U 1 1 57157BE7
 P 3350 3750
-F 0 "#PWR09" H 3350 3600 50  0001 C CNN
+F 0 "#PWR6" H 3350 3600 50  0001 C CNN
 F 1 "VDD" H 3350 3900 50  0000 C CNN
 F 2 "" H 3350 3750 50  0000 C CNN
@@
 $EndComp
 $Comp
-L VDD #PWR010
+L VDD #PWR14
 U 1 1 57157C11
 P 5200 1650
-F 0 "#PWR010" H 5200 1500 50  0001 C CNN
+F 0 "#PWR14" H 5200 1500 50  0001 C CNN
 F 1 "VDD" H 5200 1800 50  0000 C CNN
 F 2 "" H 5200 1650 50  0000 C CNN
@@
 $EndComp
 $Comp
-L VCC #PWR011
+L VCC #PWR11
 U 1 1 57157C3B
 P 4400 1650
-F 0 "#PWR011" H 4400 1500 50  0001 C CNN
+F 0 "#PWR11" H 4400 1500 50  0001 C CNN
 F 1 "VCC" H 4400 1800 50  0000 C CNN
 F 2 "" H 4400 1650 50  0000 C CNN
@@
 $EndComp
 $Comp
-L GND #PWR012
+L GND #PWR13
 U 1 1 57157C65
 P 4800 1950
-F 0 "#PWR012" H 4800 1700 50  0001 C CNN
+F 0 "#PWR13" H 4800 1700 50  0001 C CNN
 F 1 "GND" H 4800 1800 50  0000 C CNN
 F 2 "" H 4800 1950 50  0000 C CNN
@@
 $EndComp
 $Comp
-L VCC #PWR013
+L VCC #PWR19
 U 1 1 57157CA3
 P 7500 3950
-F 0 "#PWR013" H 7500 3800 50  0001 C CNN
+F 0 "#PWR19" H 7500 3800 50  0001 C CNN
 F 1 "VCC" H 7500 4100 50  0000 C CNN
 F 2 "" H 7500 3950 50  0000 C CNN
@@
 $EndComp
 $Comp
-L GND #PWR014
+L GND #PWR20
 U 1 1 57157CC6
 P 7500 5050
-F 0 "#PWR014" H 7500 4800 50  0001 C CNN
+F 0 "#PWR20" H 7500 4800 50  0001 C CNN
 F 1 "GND" H 7500 4900 50  0000 C CNN
 F 2 "" H 7500 5050 50  0000 C CNN
@@
 reset
 $Comp
-L VDD #PWR015
+L VDD #PWR4
 U 1 1 57157FD2
 P 3300 4550
-F 0 "#PWR015" H 3300 4400 50  0001 C CNN
+F 0 "#PWR4" H 3300 4400 50  0001 C CNN
 F 1 "VDD" H 3300 4700 50  0000 C CNN
 F 2 "" H 3300 4550 50  0000 C CNN
@@
 $EndComp
 $Comp
-L GND #PWR016
+L GND #PWR5
 U 1 1 57157FFE
 P 3300 4750
-F 0 "#PWR016" H 3300 4500 50  0001 C CNN
+F 0 "#PWR5" H 3300 4500 50  0001 C CNN
 F 1 "GND" H 3300 4600 50  0000 C CNN
 F 2 "" H 3300 4750 50  0000 C CNN
@@
 PILOT
 $Comp
-L GND #PWR017
+L GND #PWR27
 U 1 1 57158345
 P 8950 2600
-F 0 "#PWR017" H 8950 2350 50  0001 C CNN
+F 0 "#PWR27" H 8950 2350 50  0001 C CNN
 F 1 "GND" H 8950 2450 50  0000 C CNN
 F 2 "" H 8950 2600 50  0000 C CNN
@@
 $EndComp
 $Comp
-L GND #PWR018
+L GND #PWR22
 U 1 1 571588B4
 P 8200 3950
-F 0 "#PWR018" H 8200 3700 50  0001 C CNN
+F 0 "#PWR22" H 8200 3700 50  0001 C CNN
 F 1 "GND" H 8200 3800 50  0000 C CNN
 F 2 "" H 8200 3950 50  0000 C CNN
@@
 $EndComp
 $Comp
-L VDD #PWR019
+L VDD #PWR24
 U 1 1 57158DE8
 P 8650 4950
-F 0 "#PWR019" H 8650 4800 50  0001 C CNN
+F 0 "#PWR24" H 8650 4800 50  0001 C CNN
 F 1 "VDD" H 8650 5100 50  0000 C CNN
 F 2 "" H 8650 4950 50  0000 C CNN
@@
 	8850 5250 8850 5350
 $Comp
-L GND #PWR020
+L GND #PWR26
 U 1 1 57158E98
 P 8850 5650
-F 0 "#PWR020" H 8850 5400 50  0001 C CNN
+F 0 "#PWR26" H 8850 5400 50  0001 C CNN
 F 1 "GND" H 8850 5500 50  0000 C CNN
 F 2 "" H 8850 5650 50  0000 C CNN
@@
 $EndComp
 $Comp
-L VDD #PWR021
+L VDD #PWR23
 U 1 1 5715923F
 P 8300 2850
-F 0 "#PWR021" H 8300 2700 50  0001 C CNN
+F 0 "#PWR23" H 8300 2700 50  0001 C CNN
 F 1 "VDD" H 8300 3000 50  0000 C CNN
 F 2 "" H 8300 2850 50  0000 C CNN
@@
 Connection ~ 8750 3200
 $Comp
-L GND #PWR022
+L GND #PWR25
 U 1 1 57159508
 P 8750 3550
-F 0 "#PWR022" H 8750 3300 50  0001 C CNN
+F 0 "#PWR25" H 8750 3300 50  0001 C CNN
 F 1 "GND" H 8750 3400 50  0000 C CNN
 F 2 "" H 8750 3550 50  0000 C CNN
@@
 $EndComp
 $Comp
-L GND #PWR023
+L GND #PWR17
 U 1 1 5715A618
 P 6000 6300
-F 0 "#PWR023" H 6000 6050 50  0001 C CNN
+F 0 "#PWR17" H 6000 6050 50  0001 C CNN
 F 1 "GND" H 6000 6150 50  0000 C CNN
 F 2 "" H 6000 6300 50  0000 C CNN
@@
 RELAY_COIL
 Wire Wire Line
-	5900 6150 6000 6150
+	5400 6150 6000 6150
 $Comp
 L C C4
@@
 Connection ~ 4400 1650
 $Comp
-L GND #PWR024
+L GND #PWR12
 U 1 1 5715A9B6
 P 4400 2000
-F 0 "#PWR024" H 4400 1750 50  0001 C CNN
+F 0 "#PWR12" H 4400 1750 50  0001 C CNN
 F 1 "GND" H 4400 1850 50  0000 C CNN
 F 2 "" H 4400 2000 50  0000 C CNN
@@
 $EndComp
 $Comp
-L GND #PWR025
+L GND #PWR10
 U 1 1 5715A9FA
 P 4100 2050
-F 0 "#PWR025" H 4100 1800 50  0001 C CNN
+F 0 "#PWR10" H 4100 1800 50  0001 C CNN
 F 1 "GND" H 4100 1900 50  0000 C CNN
 F 2 "" H 4100 2050 50  0000 C CNN
@@
 Connection ~ 8150 4650
 $Comp
-L GND #PWR026
+L GND #PWR21
 U 1 1 5715B77C
 P 8150 5000
-F 0 "#PWR026" H 8150 4750 50  0001 C CNN
+F 0 "#PWR21" H 8150 4750 50  0001 C CNN
 F 1 "GND" H 8150 4850 50  0000 C CNN
 F 2 "" H 8150 5000 50  0000 C CNN
@@
 P 3650 1650
 F 0 "D1" H 3650 1750 50  0000 C CNN
-F 1 "D" H 3650 1550 50  0000 C CNN
+F 1 "1N4007" H 3650 1550 50  0000 C CNN
 F 2 "Diodes_ThroughHole:Diode_DO-41_SOD81_Horizontal_RM10" H 3650 1650 50  0001 C CNN
 F 3 "" H 3650 1650 50  0000 C CNN
@@
 	3500 1650 3150 1650
 $Comp
-L GND #PWR027
+L GND #PWR3
 U 1 1 5715C077
 P 3250 1750
-F 0 "#PWR027" H 3250 1500 50  0001 C CNN
+F 0 "#PWR3" H 3250 1500 50  0001 C CNN
 F 1 "GND" H 3250 1600 50  0000 C CNN
 F 2 "" H 3250 1750 50  0000 C CNN
@@
 Wire Wire Line
 	3200 3300 3200 3450
+$Comp
+L CONN_01X02 P5
+U 1 1 5716D762
+P 5200 6200
+F 0 "P5" H 5200 6350 50  0000 C CNN
+F 1 "RELAYCOIL" V 5300 6200 50  0000 C CNN
+F 2 "battery-dlg:CCFLHV" H 5200 6200 50  0001 C CNN
+F 3 "" H 5200 6200 50  0000 C CNN
+	1    5200 6200
+	-1   0    0    -1
+$EndComp
+Connection ~ 5900 6150
+Wire Wire Line
+	6000 6250 5400 6250
+Connection ~ 6000 6250
 $EndSCHEMATC

Commit message: switch driver chip to make bipolar pilot signal
Parts:
- removed D1, D2: 1N4007, Diodes_ThroughHole:Diode_DO-41_SOD81_Horizontal_RM10, symbol D
- removed D3: 13V ZENER, Diodes_ThroughHole:Diode_DO-41_SOD81_Horizontal_RM10, symbol ZENER
- removed U1: 7805, battery-dlg:TO220_7805, symbol 7805
- removed U2: IXDD604PI, Power_Integrations:PDIP-8, symbol IXDD604PI
- added C10, C7, C8, C9: 1uF, symbol CAPAPOL
- added D1, D2: D_Schottky, symbol D_Schottky
- added D3: 13V TVS, symbol TVS
- added K2: RELAY, symbol RELAY_2RT
- added P6: RELAY240V, battery-dlg:CCFLHV, symbol CONN_01X02
- added P7: RELAY_CTRL, battery-dlg:CCFLHV, symbol CONN_01X02
- added Q1, Q2: 2N7000, symbol FET_N
- added R1, R8: 10K, symbol R
- added R11, R12, R13: 2700, Resistors_ThroughHole:Resistor_Horizontal_RM10mm, symbol R
- added R4: 100, symbol R
- added U1: MAX232, symbol MAX232
- P2: value 12V input -> 5V input
- P5: value RELAYCOIL -> RELAY120V
- R9: renamed from R1; value 650 -> 2700
Connections:
- net labels added: +5VD, RELAY_120V, RELAY_240V
- net labels removed: RELAY, RELAY_COIL, VCC
- wire segments 37 -> 69
Other:
- note added: "+5 Volts"
- note added: "THIS CONNECTOR ACTIVATES GIANT 50A RELAY WITH 120V COIL"
- note added: "THIS RELAY CLOSES WHEN 120VAC IS READY"
- note added: "THIS RELAY CLOSES WHEN 240VAC IS READY"
- note removed: "+12V"
- note removed: "+5V"
- moved on the sheet: C5, C6, D6, P2, P4, P5, R2, R3, R5, R6, R7, R9
