File: minievse.kicad_pcb (KiCad board)
At the start: 2 copper layers, 101.6 x 50.8 mm, 54 parts, among them IC1 ATMEGA328P-P, P1 SERIAL, P2 5V input, P3 ICSP, P4 Pilot, P5 AC_GND_AC, P6 LED_STRIP, P7 RELAY_COIL, SW1 RESET_BUTTON, U1 MAX232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

Commit message: add -cache.lib and whatever else i was doing
Parts:
- renumbered REF** to W1, REF** to W2, REF** to W3, REF** to W4
Changed lines of the file:
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@@
   )
   (setup
-    (last_trace_width 0.635)
+    (last_trace_width 0.25)
     (user_trace_width 0.254)
     (user_trace_width 0.381)
@@
     (descr "Mounting Hole 3.5mm, no annular")
     (tags "mounting hole 3.5mm no annular")
-    (fp_text reference REF** (at 0 -2.54) (layer F.SilkS)
+    (fp_text reference W4 (at 0 -2.54) (layer F.SilkS)
       (effects (font (size 1 1) (thickness 0.15)))
     )
@@
     (descr "Mounting Hole 3.5mm, no annular")
     (tags "mounting hole 3.5mm no annular")
-    (fp_text reference REF** (at 0 -4.5) (layer F.SilkS)
+    (fp_text reference W3 (at 0 -4.5) (layer F.SilkS)
       (effects (font (size 1 1) (thickness 0.15)))
     )
@@
     (descr "Mounting Hole 3.5mm, no annular")
     (tags "mounting hole 3.5mm no annular")
-    (fp_text reference REF** (at 0 4.445) (layer F.SilkS)
+    (fp_text reference W1 (at 0 4.445) (layer F.SilkS)
       (effects (font (size 1 1) (thickness 0.15)))
     )
@@
     (descr "Mounting Hole 3.5mm, no annular")
     (tags "mounting hole 3.5mm no annular")
-    (fp_text reference REF** (at 0 -4.5) (layer F.SilkS)
+    (fp_text reference W2 (at 0 -4.5) (layer F.SilkS)
       (effects (font (size 1 1) (thickness 0.15)))
     )
@@
   (segment (start 121.92 55.88) (end 123.19 55.88) (width 1.016) (layer B.Cu) (net 5))
   (segment (start 86.995 66.67246) (end 86.995 63.5) (width 0.635) (layer B.Cu) (net 6))
-  (segment (start 86.995 63.5) (end 86.995 63.5) (width 0.381) (layer B.Cu) (net 6) (status C00000))
-  (segment (start 86.995 63.5) (end 90.17 67.31) (width 0.635) (layer B.Cu) (net 6) (status C00020))
+  (segment (start 86.995 63.5) (end 86.995 63.5) (width 0.381) (layer B.Cu) (net 6))
+  (segment (start 86.995 63.5) (end 90.17 67.31) (width 0.635) (layer B.Cu) (net 6) (status 20))
   (segment (start 90.17 67.31) (end 90.17 64.135) (width 0.635) (layer B.Cu) (net 6) (status 10))
   (segment (start 79.375 73.025) (end 79.375 71.755) (width 0.635) (layer B.Cu) (net 6))
@@
   (segment (start 63.5 38.735) (end 63.5 38.735) (width 0.635) (layer B.Cu) (net 18))
   (segment (start 63.5 34.29) (end 63.5 38.735) (width 0.635) (layer B.Cu) (net 18))
-  (segment (start 76.835 63.5) (end 76.835 58.42) (width 0.635) (layer B.Cu) (net 19) (status 400000))
+  (segment (start 76.835 63.5) (end 76.835 58.42) (width 0.635) (layer B.Cu) (net 19))
   (segment (start 76.835 49.53) (end 79.375 52.07) (width 0.635) (layer B.Cu) (net 19))
   (segment (start 79.375 52.07) (end 79.375 55.88) (width 0.635) (layer B.Cu) (net 19))
@@
   (segment (start 79.375 55.88) (end 76.835 58.42) (width 0.635) (layer F.Cu) (net 19))
   (via (at 76.835 58.42) (size 0.6) (drill 0.4) (layers F.Cu B.Cu) (net 19))
-  (segment (start 55.88 49.53) (end 53.34 46.99) (width 0.635) (layer B.Cu) (net 19) (status 800000))
+  (segment (start 55.88 49.53) (end 53.34 46.99) (width 0.635) (layer B.Cu) (net 19))
   (segment (start 66.04 49.53) (end 76.2 49.53) (width 0.635) (layer B.Cu) (net 19))
   (via (at 66.04 49.53) (size 0.6) (drill 0.4) (layers F.Cu B.Cu) (net 19))
@@
   (segment (start 73.66 73.66) (end 74.295 73.025) (width 1.016) (layer B.Cu) (net 22))
   (segment (start 74.295 73.025) (end 76.835 73.025) (width 1.016) (layer B.Cu) (net 22))
-  (segment (start 40.64 29.21) (end 40.64 36.83) (width 1.016) (layer B.Cu) (net 25) (status 400000))
-  (segment (start 34.29 43.18) (end 34.29 46.355) (width 1.016) (layer B.Cu) (net 25) (status 800000))
+  (segment (start 40.64 29.21) (end 40.64 36.83) (width 1.016) (layer B.Cu) (net 25))
+  (segment (start 34.29 43.18) (end 34.29 46.355) (width 1.016) (layer B.Cu) (net 25))
   (segment (start 40.64 36.83) (end 34.29 43.18) (width 1.016) (layer B.Cu) (net 25))
-  (segment (start 34.29 46.355) (end 31.115 49.53) (width 1.016) (layer B.Cu) (net 25) (status 400000))
-  (segment (start 31.115 49.53) (end 27.94 49.53) (width 1.016) (layer B.Cu) (net 25) (status 800000))
-  (segment (start 67.945 31.75) (end 67.945 29.21) (width 1.27) (layer F.Cu) (net 25) (status 400000))
-  (segment (start 42.545 27.305) (end 40.64 29.21) (width 1.27) (layer F.Cu) (net 25) (status 800000))
+  (segment (start 34.29 46.355) (end 31.115 49.53) (width 1.016) (layer B.Cu) (net 25))
+  (segment (start 31.115 49.53) (end 27.94 49.53) (width 1.016) (layer B.Cu) (net 25))
+  (segment (start 67.945 31.75) (end 67.945 29.21) (width 1.27) (layer F.Cu) (net 25))
+  (segment (start 42.545 27.305) (end 40.64 29.21) (width 1.27) (layer F.Cu) (net 25))
   (segment (start 66.04 27.305) (end 42.545 27.305) (width 1.27) (layer F.Cu) (net 25))
   (segment (start 67.945 29.21) (end 66.04 27.305) (width 1.27) (layer F.Cu) (net 25))
@@
   (segment (start 71.755 31.75) (end 67.945 29.21) (width 1.016) (layer B.Cu) (net 25))
   (segment (start 63.5 46.99) (end 63.5 49.53) (width 1.016) (layer B.Cu) (net 25))
-  (segment (start 58.42 50.8) (end 58.42 54.61) (width 1.016) (layer B.Cu) (net 25) (status 800000))
+  (segment (start 58.42 50.8) (end 58.42 54.61) (width 1.016) (layer B.Cu) (net 25))
   (segment (start 58.42 50.8) (end 58.42 50.8) (width 1.016) (layer B.Cu) (net 25))
   (segment (start 62.23 50.8) (end 58.42 50.8) (width 1.016) (layer B.Cu) (net 25))
@@
   (segment (start 116.84 33.02) (end 111.76 33.655) (width 0.635) (layer B.Cu) (net 37) (status 20))
   (segment (start 50.8 56.515) (end 50.8 57.785) (width 0.635) (layer B.Cu) (net 38))
-  (segment (start 50.8 54.61) (end 50.8 52.705) (width 0.635) (layer B.Cu) (net 38) (status 400000))
+  (segment (start 50.8 54.61) (end 50.8 52.705) (width 0.635) (layer B.Cu) (net 38))
   (segment (start 110.49 68.58) (end 105.41 68.58) (width 0.635) (layer B.Cu) (net 38))
   (segment (start 83.82 67.31) (end 85.725 69.85) (width 0.635) (layer F.Cu) (net 38))
@@
   (segment (start 50.8 57.785) (end 45.085 64.135) (width 0.635) (layer B.Cu) (net 38) (status 20))
   (segment (start 45.085 64.135) (end 43.18 64.135) (width 0.635) (layer B.Cu) (net 38) (status 20))
-  (segment (start 42.545 73.025) (end 42.545 71.12) (width 0.635) (layer B.Cu) (net 39) (status 400000))
-  (segment (start 50.165 60.96) (end 55.88 55.245) (width 0.635) (layer B.Cu) (net 39) (status 800000))
+  (segment (start 42.545 73.025) (end 42.545 71.12) (width 0.635) (layer B.Cu) (net 39))
+  (segment (start 50.165 60.96) (end 55.88 55.245) (width 0.635) (layer B.Cu) (net 39))
   (segment (start 50.165 63.5) (end 50.165 60.96) (width 0.635) (layer B.Cu) (net 39))
   (segment (start 48.26 65.405) (end 50.165 63.5) (width 0.635) (layer B.Cu) (net 39))
@@
   (via (at 45.72 67.945) (size 0.6) (drill 0.4) (layers F.Cu B.Cu) (net 39))
   (segment (start 42.545 71.12) (end 45.72 67.945) (width 0.635) (layer B.Cu) (net 39))
-  (segment (start 55.88 55.245) (end 55.88 54.61) (width 0.635) (layer B.Cu) (net 39) (status C00000))
+  (segment (start 55.88 55.245) (end 55.88 54.61) (width 0.635) (layer B.Cu) (net 39))
   (segment (start 103.505 53.975) (end 103.505 53.975) (width 0.25) (layer B.Cu) (net 41) (status 30))
   (segment (start 79.375 50.165) (end 76.2 46.99) (width 0.381) (layer B.Cu) (net 41))
