File: minievse.sch (KiCad schematic (older format))
At the start: 60 parts, among them IC1 ATMEGA328P-P, P1 SERIAL, P2 5V input, P3 ICSP, P4 Pilot, P5 AC_GND_AC, P6 LED_STRIP, P7 RELAY_COIL, Q1 FET_N, Q2 FET_P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

Commit message: add -cache.lib and whatever else i was doing
Parts:
- added W1, W2, W3, W4: TEST_1P, Mounting_Holes:MountingHole_3.5mm, symbol TEST_1P
- C7: value C -> 104; footprint (none) -> Capacitors_ThroughHole:C_Disc_D3_P2.5
- L1, L2: footprint (none) -> Inductors:INDUCTOR_V
- Q1: footprint (none) -> ~; symbol FET_N -> Q_NMOS_GDS
- R12, R13, R22: footprint (none) -> Resistors_ThroughHole:Resistor_Horizontal_RM10mm
Connections:
- net BOOST12: no longer Q1.D
- net BOOST5: no longer Q1.G
- net GND: no longer Q1.S
Changed lines of the file:
@@
 Connection ~ 6350 5650
 $Comp
-L FET_N Q1
+L Q_NMOS_GDS Q1
 U 1 1 5732510A
 P 6800 2000
-F 0 "Q1" H 6900 2000 50  0000 C CNN
+F 0 "Q1" H 7050 2000 50  0000 C CNN
 F 1 "FET_N" H 6653 1753 50  0000 C CNN
-F 2 "" H 6800 2000 60  0000 C CNN
+F 2 "~" H 6800 2000 60  0001 C CNN
 F 3 "" H 6800 2000 60  0000 C CNN
 	1    6800 2000
@@
 F 0 "L1" V 6600 1550 50  0000 C CNN
 F 1 "INDUCTOR" V 6750 1550 50  0000 C CNN
-F 2 "" H 6650 1550 50  0000 C CNN
+F 2 "Inductors:INDUCTOR_V" H 6650 1550 50  0001 C CNN
 F 3 "" H 6650 1550 50  0000 C CNN
 	1    6650 1550
@@
 F 0 "L2" V 7650 2350 50  0000 C CNN
 F 1 "INDUCTOR" V 7800 2350 50  0000 C CNN
-F 2 "" H 7700 2350 50  0000 C CNN
+F 2 "Inductors:INDUCTOR_V" H 7700 2350 50  0001 C CNN
 F 3 "" H 7700 2350 50  0000 C CNN
 	1    7700 2350
@@
 Text Label 5800 1750 2    60   ~ 0
 +2.5V
-$Comp
-L C C7
-U 1 1 573299A8
-P 5550 1900
-F 0 "C7" H 5575 2000 50  0000 L CNN
-F 1 "C" H 5575 1800 50  0000 L CNN
-F 2 "" H 5588 1750 50  0000 C CNN
-F 3 "" H 5550 1900 50  0000 C CNN
-	1    5550 1900
-	1    0    0    -1
-$EndComp
 Wire Wire Line
 	5550 1750 5800 1750
@@
 F 0 "R13" V 5880 1900 50  0000 C CNN
 F 1 "10K" V 5800 1900 50  0000 C CNN
-F 2 "" V 5730 1900 50  0000 C CNN
+F 2 "Resistors_ThroughHole:Resistor_Horizontal_RM10mm" V 5730 1900 50  0001 C CNN
 F 3 "" H 5800 1900 50  0000 C CNN
 	1    5800 1900
@@
 F 0 "R12" V 5880 1500 50  0000 C CNN
 F 1 "10K" V 5800 1500 50  0000 C CNN
-F 2 "" V 5730 1500 50  0000 C CNN
+F 2 "Resistors_ThroughHole:Resistor_Horizontal_RM10mm" V 5730 1500 50  0001 C CNN
 F 3 "" H 5800 1500 50  0000 C CNN
 	1    5800 1500
@@
 F 0 "R22" V 8280 1300 50  0000 C CNN
 F 1 "22" V 8200 1300 50  0000 C CNN
-F 2 "" V 8130 1300 50  0000 C CNN
+F 2 "Resistors_ThroughHole:Resistor_Horizontal_RM10mm" V 8130 1300 50  0001 C CNN
 F 3 "" H 8200 1300 50  0000 C CNN
 	1    8200 1300
@@
 	8050 1300 6950 1300
 $Comp
-L -12VA #PWR?
+L -12VA #PWR047
 U 1 1 5732BF7E
 P 7450 4250
-F 0 "#PWR?" H 7450 4100 50  0001 C CNN
+F 0 "#PWR047" H 7450 4100 50  0001 C CNN
 F 1 "-12VA" H 7450 4390 50  0000 C CNN
 F 2 "" H 7450 4250 50  0000 C CNN
@@
 	-1   0    0    1
 $EndComp
+$Comp
+L TEST_1P W1
+U 1 1 5732CC80
+P 1700 1300
+F 0 "W1" H 1700 1570 50  0000 C CNN
+F 1 "TEST_1P" H 1700 1500 50  0000 C CNN
+F 2 "Mounting_Holes:MountingHole_3.5mm" H 1900 1300 50  0001 C CNN
+F 3 "" H 1900 1300 50  0000 C CNN
+	1    1700 1300
+	1    0    0    -1
+$EndComp
+$Comp
+L TEST_1P W2
+U 1 1 5732D197
+P 1700 1650
+F 0 "W2" H 1700 1920 50  0000 C CNN
+F 1 "TEST_1P" H 1700 1850 50  0000 C CNN
+F 2 "Mounting_Holes:MountingHole_3.5mm" H 1900 1650 50  0001 C CNN
+F 3 "" H 1900 1650 50  0000 C CNN
+	1    1700 1650
+	1    0    0    -1
+$EndComp
+$Comp
+L TEST_1P W3
+U 1 1 5732D26E
+P 1700 2000
+F 0 "W3" H 1700 2270 50  0000 C CNN
+F 1 "TEST_1P" H 1700 2200 50  0000 C CNN
+F 2 "Mounting_Holes:MountingHole_3.5mm" H 1900 2000 50  0001 C CNN
+F 3 "" H 1900 2000 50  0000 C CNN
+	1    1700 2000
+	1    0    0    -1
+$EndComp
+$Comp
+L TEST_1P W4
+U 1 1 5732D4D4
+P 1700 2350
+F 0 "W4" H 1700 2620 50  0000 C CNN
+F 1 "TEST_1P" H 1700 2550 50  0000 C CNN
+F 2 "Mounting_Holes:MountingHole_3.5mm" H 1900 2350 50  0001 C CNN
+F 3 "" H 1900 2350 50  0000 C CNN
+	1    1700 2350
+	1    0    0    -1
+$EndComp
+$Comp
+L C C7
+U 1 1 5732DD49
+P 5550 1900
+F 0 "C7" H 5575 2000 50  0000 L CNN
+F 1 "104" H 5575 1800 50  0000 L CNN
+F 2 "Capacitors_ThroughHole:C_Disc_D3_P2.5" H 5588 1750 50  0001 C CNN
+F 3 "" H 5550 1900 50  0000 C CNN
+	1    5550 1900
+	1    0    0    -1
+$EndComp
 $EndSCHEMATC
